Commit message: update to 6dof arm

File: urdf/arm.xacro (robot description, xacro)
@@ -49,17 +49,16 @@
     <xacro:cylinder_link name="link3" length="0.145" radius="0.025" color="1 0 0 1" xyz="0 0 0.0725"/>
     <xacro:revolute_joint name="joint3" parent="link2" child="link3" xyz="0 0 0.105" axis="0 1 0" lower="-1.57" upper="1.57"/>
-    <xacro:cylinder_link name="link4" length="0.065" radius="0.025" color="1 0 1 1" xyz="0 0 0.0325"/>
-    <xacro:revolute_joint name="joint4" parent="link3" child="link4" xyz="0 0 0.145" axis="0 1 0" lower="-1.57" upper="1.57"/>
-    <xacro:cylinder_link name="link5" length="0.03" radius="0.015" color="1 1 0 1" xyz="0 0 0.015"/>
-    <xacro:revolute_joint name="joint5" parent="link4" child="link5" xyz="0 0 0.065" axis="0 0 1" lower="-1.57" upper="1.57"/>
-    <!-- <xacro:cylinder-link name="claw_link" length="0.4" radius="0.1" color="0 1 1 1" xyz="0 0 0.2"/> -->
+    <xacro:cylinder_link name="link4" length="0.02" radius="0.025" color="1 0 1 1" xyz="0 0.025 0.005"/>
+    <xacro:revolute_joint name="joint4" parent="link3" child="link4" xyz="0 0.025 0.145" axis="0 1 0" lower="-1.57" upper="1.57"/>
+    <xacro:cylinder_link name="link5" length="0.07" radius="0.015" color="1 1 1 1" xyz="0 0 0.03"/>
+    <xacro:revolute_joint name="joint5" parent="link4" child="link5" xyz="0 0.025 0.02" axis="1 0 0" lower="-1.57" upper="1.57"/>
     <link name="gripper_base">
-        <inertial>
+        <!-- <inertial>
             <origin xyz="0 0 0"/>
             <mass value="0.5"/>
             <inertia ixx="0.005" ixy="0" ixz="0" iyy="0.005" iyz="0" izz="0.005"/>
-        </inertial>
+        </inertial> -->
         <visual>
-            <origin xyz="0 0 0.0125" rpy="0 0 0"/>
+            <origin xyz="0 0 0.0175" rpy="0 0 0"/>
             <geometry>
                 <box size="0.025 0.055 0.025"/>
@@ -91,13 +90,17 @@
         <origin xyz="0 0 0.0125" rpy="0 0 0"/>
     </joint>
-    <xacro:revolute_joint name="joint6" parent="link5" child="gripper_base" xyz="0 0 0.03" axis="1 0 0" lower="-1.57" upper="1.57"/>
+    <joint name="joint7" type="fixed">
+        <parent link="link5"/>
+        <child link="gripper_base"/>
+        <origin xyz="0 0 0.06" rpy="0 0 0"/>
+    </joint>
     <link name="left_finger">
         <visual>
-            <origin xyz="0 0.015 0.0425" rpy="0 0 0"/>
+            <origin xyz="0 0.02 0.05" rpy="0 0 0"/>
             <geometry>
                 <box size="0.01 0.01 0.085"/>
             </geometry>
             <material name="red">
-                <color rgba="1 0 0 1"/>
+                <color rgba="1 0.65 0 1"/>
             </material>
         </visual>
@@ -109,11 +112,14 @@
         </collision>
     </link>
-    <joint name="left_finger_joint" type="fixed">
+    <joint name="left_finger_joint" type="prismatic">
         <parent link="gripper_base"/>
         <child link="left_finger"/>
+        <origin xyz="0 0 0" rpy="0 0 0"/>
+        <axis xyz="0 1 0"/>
+        <limit lower="-0.015" upper="0" effort="10" velocity="1"/>
     </joint>
     <link name="right_finger">
         <visual>
-            <origin xyz="0 -0.015 0.0425" rpy="0 0 0"/>
+            <origin xyz="0 -0.02 0.05" rpy="0 0 0"/>
             <geometry>
                 <box size="0.01 0.01 0.085"/>
@@ -130,7 +136,11 @@
         </collision>
     </link>
-    <joint name="right_finger_joint" type="fixed">
+    <joint name="right_finger_joint" type="prismatic">
         <parent link="gripper_base"/>
         <child link="right_finger"/>
+        <origin xyz="0 0 0" rpy="0 0 0"/>
+        <axis xyz="0 1 0"/>
+        <limit lower="0" upper="0.015" effort="10" velocity="1"/>
+        <mimic joint="left_finger_joint" multiplier="-1" offset="0"/>
     </joint>
     <ros2_control name="ArmSystem" type="system">

Commit message: update to 6dof arm

File: urdf/arm.xacro (robot description, xacro)
@@ -90,5 +90,5 @@
         <origin xyz="0 0 0.0125" rpy="0 0 0"/>
     </joint>
-    <joint name="joint7" type="fixed">
+    <joint name="joint6" type="fixed">
         <parent link="link5"/>
         <child link="gripper_base"/>

Commit message: joint 6 fixed -> revolute

File: urdf/arm.xacro (robot description, xacro)
@@ -4,9 +4,9 @@
     <xacro:macro name="cylinder_link" params="name length radius color xyz">
         <link name="${name}">
-            <inertial>
+            <!-- <inertial>
                 <origin xyz="0 0 0"/>
                 <mass value="1.0"/>
                 <inertia ixx="0.01" ixy="0" ixz="0" iyy="0.01" iyz="0" izz="0.01"/>
-            </inertial>
+            </inertial> -->
             <visual>
                 <origin xyz="${xyz}" rpy="0 0 0"/>
@@ -76,5 +76,5 @@
     </link>
     <link name="end_effector_link">
-        <inertial>
+        <!-- <inertial>
             <origin xyz="0 0 0"/>
             <mass value="0.1"/>
@@ -83,5 +83,5 @@
                 iyy="0.001" iyz="0"
                 izz="0.001"/>
-        </inertial>
+        </inertial> -->
     </link>
     <joint name="ee_fixed" type="fixed">
@@ -90,9 +90,5 @@
         <origin xyz="0 0 0.0125" rpy="0 0 0"/>
     </joint>
-    <joint name="joint6" type="fixed">
-        <parent link="link5"/>
-        <child link="gripper_base"/>
-        <origin xyz="0 0 0.06" rpy="0 0 0"/>
-    </joint>
+    <xacro:revolute_joint name="joint6" parent="link5" child="gripper_base" xyz="0 0 0.06" axis="0 0 1" lower="-1.57" upper="1.57"/>
     <link name="left_finger">
         <visual>
